Commit message: Update Gazebo launch file and add RViz configuration
- Updated the latest build timestamp in the log file.
- Modified the gazebo.launch.py file to:
  - Remove unnecessary imports and comments.
  - Add RViz node configuration to launch RViz with the specified configuration file.
- Added a .gitignore file to exclude common build artifacts and local configuration files from version control.

File: hcr5_ws/install/hcr5_description/share/hcr5_description/urdf/hcr5.xacro (robot description, xacro)
@@ -1 +1,289 @@
-/home/forsaken/Documents/hcr5_ws/src/hcr5_description/urdf/hcr5.xacro
+<?xml version="1.0"?>
+<robot name="hcr5" xmlns:xacro="http://www.ros.org/wiki/xacro">
+<xacro:include filename="$(find hcr5_description)/urdf/materials.xacro" />
+<!-- <xacro:include filename="$(find hcr5_description)/urdf/hcr5.trans" /> -->
+<xacro:include filename="$(find hcr5_description)/urdf/hcr5.gazebo" />
+<xacro:arg name="use_mock_hardware" default="true" />
+<link name="world"/>
+<joint name="world_joint" type="fixed">
+  <parent link="world"/>
+  <child link="base_link"/>
+  <origin xyz="0 0 0" rpy="0 0 0"/>
+</joint>
+<link name="base_link">
+  <inertial>
+    <origin xyz="0.044693591972953806 -9.689819846991377e-05 0.013982771179495564" rpy="0 0 0"/>
+    <mass value="4.071462983655495"/>
+    <inertia ixx="0.004614" iyy="0.063084" izz="0.067151" ixy="-2e-05" iyz="0.0" ixz="-0.000189"/>
+  </inertial>
+  <visual>
+    <origin xyz="0 0 0" rpy="0 0 0"/>
+    <geometry>
+      <mesh filename="package://hcr5_description/meshes/base_link.stl" scale="0.001 0.001 0.001"/>
+    </geometry>
+    <material name="grey">
+      <color rgba="0.5 0.5 0.5 1.0"/>
+    </material>
+  </visual>
+  <collision>
+    <origin xyz="0 0 0" rpy="0 0 0"/>
+    <geometry>
+      <mesh filename="package://hcr5_description/meshes/base_link.stl" scale="0.001 0.001 0.001"/>
+    </geometry>
+  </collision>
+</link>
+<link name="link1_1">
+  <inertial>
+    <origin xyz="-0.009232924655966162 5.611908895686318e-08 0.08981078121700108" rpy="0 0 0"/>
+    <mass value="17.125748524580114"/>
+    <inertia ixx="0.054601" iyy="0.061186" izz="0.036738" ixy="0.0" iyz="-0.0" ixz="0.004569"/>
+  </inertial>
+  <visual>
+    <origin xyz="-0.0 0.0 -0.03" rpy="0 0 0"/>
+    <geometry>
+      <mesh filename="package://hcr5_description/meshes/link1_1.stl" scale="0.001 0.001 0.001"/>
+    </geometry>
+    <material name="grey">
+      <color rgba="0.5 0.5 0.5 1.0"/>
+    </material>
+  </visual>
+  <collision>
+    <origin xyz="-0.0 0.0 -0.03" rpy="0 0 0"/>
+    <geometry>
+      <mesh filename="package://hcr5_description/meshes/link1_1.stl" scale="0.001 0.001 0.001"/>
+    </geometry>
+  </collision>
+</link>
+<link name="link2_1">
+  <inertial>
+    <origin xyz="-0.08134423156498356 0.0004999972193747809 0.21200027982915884" rpy="0 0 0"/>
+    <mass value="32.073698785630135"/>
+    <inertia ixx="1.334728" iyy="1.368804" izz="0.0845" ixy="-5e-06" iyz="-0.003172" ixz="-0.002068"/>
+  </inertial>
+  <visual>
+    <origin xyz="0.0785 0.0 -0.148778" rpy="0 0 0"/>
+    <geometry>
+      <mesh filename="package://hcr5_description/meshes/link2_1.stl" scale="0.001 0.001 0.001"/>
+    </geometry>
+    <material name="grey">
+      <color rgba="0.5 0.5 0.5 1.0"/>
+    </material>
+  </visual>
+  <collision>
+    <origin xyz="0.0785 0.0 -0.148778" rpy="0 0 0"/>
+    <geometry>
+      <mesh filename="package://hcr5_description/meshes/link2_1.stl" scale="0.001 0.001 0.001"/>
+    </geometry>
+  </collision>
+</link>
+<link name="link3_1">
+  <inertial>
+    <origin xyz="0.03733088153046067 -8.45436915776097e-06 0.32700293666580915" rpy="0 0 0"/>
+    <mass value="6.636542484506931"/>
+    <inertia ixx="0.008668" iyy="0.014027" izz="0.010649" ixy="-0.0" iyz="0.0" ixz="0.001661"/>
+  </inertial>
+  <visual>
+    <origin xyz="0.077848 -0.001 -0.572778" rpy="0 0 0"/>
+    <geometry>
+      <mesh filename="package://hcr5_description/meshes/link3_1.stl" scale="0.001 0.001 0.001"/>
+    </geometry>
+    <material name="orange">
+      <color rgba="1.0 0.5 0.0 1.0"/>
+    </material>
+  </visual>
+  <collision>
+    <origin xyz="0.077848 -0.001 -0.572778" rpy="0 0 0"/>
+    <geometry>
+      <mesh filename="package://hcr5_description/meshes/link3_1.stl" scale="0.001 0.001 0.001"/>
+    </geometry>
+  </collision>
+</link>
+<link name="link4_1">
+  <inertial>
+    <origin xyz="-0.053462210233883714 -3.2261679182082545e-07 0.022076827880824546" rpy="0 0 0"/>
+    <mass value="6.518501202798632"/>
+    <inertia ixx="0.011005" iyy="0.012783" izz="0.007491" ixy="-0.0" iyz="0.0" ixz="0.001222"/>
+  </inertial>
+  <visual>
+    <origin xyz="0.107864 -0.000992 -0.911345" rpy="0 0 0"/>
+    <geometry>
+      <mesh filename="package://hcr5_description/meshes/link4_1.stl" scale="0.001 0.001 0.001"/>
+    </geometry>
+    <material name="orange">
+      <color rgba="1.0 0.5 0.0 1.0"/>
+    </material>
+  </visual>
+  <collision>
+    <origin xyz="0.107864 -0.000992 -0.911345" rpy="0 0 0"/>
+    <geometry>
+      <mesh filename="package://hcr5_description/meshes/link4_1.stl" scale="0.001 0.001 0.001"/>
+    </geometry>
+  </collision>
+</link>
+<link name="link5_1">
+  <inertial>
+    <origin xyz="-0.022082116809040042 -5.860596366637823e-07 0.0534553107989999" rpy="0 0 0"/>
+    <mass value="6.518501237017786"/>
+    <inertia ixx="0.007541" iyy="0.012794" izz="0.010966" ixy="0.0" iyz="-0.0" ixz="0.001224"/>
+  </inertial>
+  <visual>
+    <origin xyz="0.169864 -0.000992 -1.000941" rpy="0 0 0"/>
+    <geometry>
+      <mesh filename="package://hcr5_description/meshes/link5_1.stl" scale="0.001 0.001 0.001"/>
+    </geometry>
+    <material name="orange">
+     <color rgba="1.0 0.5 0.0 1.0"/>
+    </material>
+  </visual>
+  <collision>
+    <origin xyz="0.169864 -0.000992 -1.000941" rpy="0 0 0"/>
+    <geometry>
+      <mesh filename="package://hcr5_description/meshes/link5_1.stl" scale="0.001 0.001 0.001"/>
+    </geometry>
+  </collision>
+</link>
+<link name="link6_1">
+  <inertial>
+    <origin xyz="-0.019264152679962065 -4.5474100852818493e-07 -0.0005907014657897669" rpy="0 0 0"/>
+    <mass value="1.6914762668461325"/>
+    <inertia ixx="0.001473" iyy="0.00094" izz="0.000976" ixy="0.0" iyz="0.0" ixz="-8e-06"/>
+  </inertial>
+  <visual>
+    <origin xyz="0.25946 -0.000992 -1.062941" rpy="0 0 0"/>
+    <geometry>
+      <mesh filename="package://hcr5_description/meshes/link6_1.stl" scale="0.001 0.001 0.001"/>
+    </geometry>
+    <material name="silver">
+      <color rgba="0.7 0.7 0.7 1.0"/>
+    </material>
+  </visual>
+  <collision>
+    <origin xyz="0.25946 -0.000992 -1.062941" rpy="0 0 0"/>
+    <geometry>
+      <mesh filename="package://hcr5_description/meshes/link6_1.stl" scale="0.001 0.001 0.001"/>
+    </geometry>
+  </collision>
+</link>
+<joint name="joint_1" type="revolute">
+  <origin xyz="0.0 0.0 0.03" rpy="0 0 0"/>
+  <parent link="base_link"/>
+  <child link="link1_1"/>
+  <axis xyz="0.0 -0.0 1.0"/>
+  <limit upper="6.283185" lower="0.0" effort="1000" velocity="100"/>
+</joint>
+<joint name="joint_2" type="revolute">
+  <origin xyz="-0.0785 0.0 0.118778" rpy="0 0 0"/>
+  <parent link="link1_1"/>
+  <child link="link2_1"/>
+  <axis xyz="-1.0 0.0 0.0"/>
+  <limit upper="1.570796" lower="-1.570796" effort="2000" velocity="100"/>
+</joint>
+<joint name="joint_3" type="revolute">
+  <origin xyz="0.000652 0.001 0.424" rpy="0 0 0"/>
+  <parent link="link2_1"/>
+  <child link="link3_1"/>
+  <axis xyz="1.0 0.0 0.0"/>
+  <limit upper="2.268928" lower="-2.268928" effort="1000" velocity="100"/>
+</joint>
+<joint name="joint_4" type="revolute">
+  <origin xyz="-0.030016 -8e-06 0.338567" rpy="0 0 0"/>
+  <parent link="link3_1"/>
+  <child link="link4_1"/>
+  <axis xyz="-1.0 0.0 -0.0"/>
+  <limit upper="2.96706" lower="-2.96706" effort="1000" velocity="100"/>
+</joint>
+<joint name="joint_5" type="revolute">
+  <origin xyz="-0.062 0.0 0.089596" rpy="0 0 0"/>
+  <parent link="link4_1"/>
+  <child link="link5_1"/>
+  <axis xyz="-0.0 -0.0 1.0"/>
+  <limit upper="2.094395" lower="-2.094395" effort="1000" velocity="100"/>
+</joint>
+<joint name="joint_6" type="revolute">
+  <origin xyz="-0.089596 0.0 0.062" rpy="0 0 0"/>
+  <parent link="link5_1"/>
+  <child link="link6_1"/>
+  <axis xyz="-1.0 -0.0 0.0"/>
+  <limit upper="6.283185" lower="0.0" effort="1000" velocity="100"/>
+</joint>
+<ros2_control name="HCR5_Control" type="system">
+  <hardware>
+    <xacro:if value="$(arg use_mock_hardware)">
+      <plugin>gz_ros2_control/GazeboSimSystem</plugin>
+    </xacro:if>
+    <xacro:unless value="$(arg use_mock_hardware)">
+      <plugin>hcr_hardware/HCR5HardwareInterface</plugin>
+      <param name="robot_ip">192.168.1.10</param>
+    </xacro:unless>
+  </hardware>
+  <joint name="joint_1">
+    <command_interface name="position"/>
+    <state_interface name="position"/>
+    <state_interface name="velocity"/>
+  </joint>
+  <joint name="joint_2">
+    <command_interface name="position"/>
+    <state_interface name="position"/>
+    <state_interface name="velocity"/>
+  </joint>
+  <joint name="joint_3">
+    <command_interface name="position"/>
+    <state_interface name="position"/>
+    <state_interface name="velocity"/>
+  </joint>
+  <joint name="joint_4">
+    <command_interface name="position"/>
+    <state_interface name="position"/>
+    <state_interface name="velocity"/>
+  </joint>
+  <joint name="joint_5">
+    <command_interface name="position"/>
+    <state_interface name="position"/>
+    <state_interface name="velocity"/>
+  </joint>
+  <joint name="joint_6">
+    <command_interface name="position"/>
+    <state_interface name="position"/>
+    <state_interface name="velocity"/>
+  </joint>
+</ros2_control>
+<gazebo>
+  <plugin filename="gz_ros2_control-system" name="gz_ros2_control::GazeboSimROS2ControlPlugin">
+    <parameters>$(find hcr5_description)/config/hcr5_controllers.yaml</parameters>
+  </plugin>
+  <plugin
+    filename="gz-sim-sensors-system"
+    name="gz::sim::systems::Sensors">
+    <render_engine>ogre2</render_engine>
+  </plugin>
+</gazebo>
+<link name="camera_link">
+    <visual>
+      <geometry>
+        <box size="0.02 0.05 0.02"/>
+      </geometry>
+      <material name="red">
+        <color rgba="1 0 0 1"/>
+      </material>
+    </visual>
+  </link>
+  <joint name="camera_joint" type="fixed">
+    <parent link="link6_1"/> <child link="camera_link"/>
+    <origin xyz="-0.053 0.0 0.0" rpy="3.14159 3.14159 0.0"/>
+  </joint>
+<gazebo reference="camera_link">
+  <sensor name="robot_camera" type="camera">
+    <topic>camera/image_raw</topic>
+    <camera>
+      <horizontal_fov>1.089</horizontal_fov>
+      <image>
+        <width>640</width>
+        <height>480</height>
+      </image>
+    </camera>
+    <always_on>1</always_on>
+    <update_rate>30</update_rate>
+    <visualize>true</visualize>
+  </sensor>
+</gazebo>
+</robot>

File: hcr5_ws/install/hcr5_description/share/hcr5_description/urdf/materials.xacro (robot description, xacro)
@@ -1 +1,9 @@
-/home/forsaken/Documents/hcr5_ws/src/hcr5_description/urdf/materials.xacro
+<robot xmlns:xacro="http://www.ros.org/wiki/xacro">
+  <gazebo reference="base_link"><material>Gazebo/Black</material></gazebo>
+  <gazebo reference="link1_1"><material>Gazebo/Black</material></gazebo>
+  <gazebo reference="link2_1"><material>Gazebo/Black</material></gazebo>
+  <gazebo reference="link3_1"><material>Gazebo/Orange</material></gazebo>
+  <gazebo reference="link4_1"><material>Gazebo/Orange</material></gazebo>
+  <gazebo reference="link5_1"><material>Gazebo/Orange</material></gazebo>
+  <gazebo reference="link6_1"><material>Gazebo/Grey</material></gazebo>
+</robot>

Commit message: Add camera pole and update camera link in URDF for improved visualization

File: hcr5_ws/install/hcr5_description/share/hcr5_description/urdf/hcr5.xacro (robot description, xacro)
@@ -258,26 +258,72 @@
   </plugin>
 </gazebo>
+<link name="camera_pole">
+  <visual>
+    <geometry>
+      <cylinder radius="0.03" length="2.0"/>
+    </geometry>
+    <material name="gray">
+      <color rgba="0.5 0.5 0.5 1.0"/>
+    </material>
+  </visual>
+  <collision>
+    <geometry>
+      <cylinder radius="0.03" length="2.0"/>
+    </geometry>
+  </collision>
+</link>
+<joint name="world_to_pole" type="fixed">
+  <parent link="base_link"/>
+  <child link="camera_pole"/>
+  <origin xyz="1.0 1.0 1.0" rpy="0 0 0"/> </joint>
 <link name="camera_link">
-    <visual>
-      <geometry>
-        <box size="0.02 0.05 0.02"/>
-      </geometry>
-      <material name="red">
-        <color rgba="1 0 0 1"/>
-      </material>
-    </visual>
-  </link>
-  <joint name="camera_joint" type="fixed">
-    <parent link="link6_1"/> <child link="camera_link"/>
-    <origin xyz="-0.053 0.0 0.0" rpy="3.14159 3.14159 0.0"/>
-  </joint>
+  <visual>
+    <geometry>
+      <box size="0.05 0.05 0.05"/>
+    </geometry>
+    <material name="blue">
+      <color rgba="0 0 1 1"/>
+    </material>
+  </visual>
+</link>
+<joint name="pole_to_camera" type="fixed">
+  <parent link="camera_pole"/>
+  <child link="camera_link"/>
+  <origin xyz="0 0 1.0" rpy="0 0.785 3.925"/>
+</joint>
+<!-- <gazebo reference="camera_link">
+  <sensor name="external_camera" type="camera">
+    <update_rate>30.0</update_rate>
+    <camera name="head">
+      <horizontal_fov>1.3962634</horizontal_fov>
+      <image>
+        <width>800</width>
+        <height>800</height>
+        <format>R8G8B8</format>
+      </image>
+      <clip>
+        <near>0.02</near>
+        <far>300</far>
+      </clip>
+    </camera>
+    <plugin name="camera_controller" filename="libgazebo_ros_camera.so">
+      <alwaysOn>true</alwaysOn>
+      <updateRate>0.0</updateRate>
+      <cameraName>external_camera</cameraName>
+      <imageTopicName>image_raw</imageTopicName>
+      <cameraInfoTopicName>camera_info</cameraInfoTopicName>
+      <frameName>camera_link</frameName>
+    </plugin>
+  </sensor>
+</gazebo> -->
 <gazebo reference="camera_link">
-  <sensor name="robot_camera" type="camera">
+  <sensor name="external_camera" type="camera">
     <topic>camera/image_raw</topic>
     <camera>
       <horizontal_fov>1.089</horizontal_fov>
       <image>
-        <width>640</width>
-        <height>480</height>
+        <width>1280</width>
+        <height>720</height>
+        <format>R8G8B8</format>
       </image>
     </camera>
@@ -285,4 +331,12 @@
     <update_rate>30</update_rate>
     <visualize>true</visualize>
+    <plugin name="camera_controller" filename="libgazebo_ros_camera.so">
+      <alwaysOn>true</alwaysOn>
+      <updateRate>0.0</updateRate>
+      <cameraName>external_camera</cameraName>
+      <imageTopicName>image_raw</imageTopicName>
+      <cameraInfoTopicName>camera_info</cameraInfoTopicName>
+      <frameName>camera_link</frameName>
+    </plugin>
   </sensor>
 </gazebo>

Commit message: Refactor camera setup in URDF and launch files for dual camera support

File: hcr5_ws/install/hcr5_description/share/hcr5_description/urdf/hcr5.xacro (robot description, xacro)
@@ -258,8 +258,8 @@
   </plugin>
 </gazebo>
-<link name="camera_pole">
-  <visual>
-    <geometry>
-      <cylinder radius="0.03" length="2.0"/>
+<link name="camera_pole1">
+  <visual>
+    <geometry>
+      <cylinder radius="0.02" length="2.0"/>
     </geometry>
     <material name="gray">
@@ -269,13 +269,34 @@
   <collision>
     <geometry>
-      <cylinder radius="0.03" length="2.0"/>
-    </geometry>
-  </collision>
-</link>
-<joint name="world_to_pole" type="fixed">
+      <cylinder radius="0.02" length="2.0"/>
+    </geometry>
+  </collision>
+</link>
+<link name="camera_pole2">
+  <visual>
+    <geometry>
+      <cylinder radius="0.02" length="2.0"/>
+    </geometry>
+    <material name="gray">
+      <color rgba="0.5 0.5 0.5 1.0"/>
+    </material>
+  </visual>
+  <collision>
+    <geometry>
+      <cylinder radius="0.02" length="2.0"/>
+    </geometry>
+  </collision>
+</link>
+<joint name="world_to_pole1" type="fixed">
   <parent link="base_link"/>
-  <child link="camera_pole"/>
-  <origin xyz="1.0 1.0 1.0" rpy="0 0 0"/> </joint>
-<link name="camera_link">
+  <child link="camera_pole1"/>
+  <origin xyz="1.0 1.0 1.0" rpy="0 0 0"/>
+</joint>
+<joint name="world_to_pole2" type="fixed">
+  <parent link="base_link"/>
+  <child link="camera_pole2"/>
+  <origin xyz="-1.0 -1.0 1.0" rpy="0 0 0"/>
+</joint>
+<link name="camera_link1">
   <visual>
     <geometry>
@@ -287,43 +308,31 @@
   </visual>
 </link>
-<joint name="pole_to_camera" type="fixed">
-  <parent link="camera_pole"/>
-  <child link="camera_link"/>
-  <origin xyz="0 0 1.0" rpy="0 0.785 3.925"/>
-</joint>
-<!-- <gazebo reference="camera_link">
-  <sensor name="external_camera" type="camera">
-    <update_rate>30.0</update_rate>
-    <camera name="head">
-      <horizontal_fov>1.3962634</horizontal_fov>
-      <image>
-        <width>800</width>
-        <height>800</height>
-        <format>R8G8B8</format>
-      </image>
-      <clip>
-        <near>0.02</near>
-        <far>300</far>
-      </clip>
-    </camera>
-    <plugin name="camera_controller" filename="libgazebo_ros_camera.so">
-      <alwaysOn>true</alwaysOn>
-      <updateRate>0.0</updateRate>
-      <cameraName>external_camera</cameraName>
-      <imageTopicName>image_raw</imageTopicName>
-      <cameraInfoTopicName>camera_info</cameraInfoTopicName>
-      <frameName>camera_link</frameName>
-    </plugin>
-  </sensor>
-</gazebo> -->
-<gazebo reference="camera_link">
-  <sensor name="external_camera" type="camera">
-    <topic>camera/image_raw</topic>
-    <camera>
+<link name="camera_link2">
+  <visual>
+    <geometry>
+      <box size="0.05 0.05 0.05"/>
+    </geometry>
+    <material name="blue">
+      <color rgba="0 0 1 1"/>
+    </material>
+  </visual>
+</link>
+<joint name="pole_to_camera1" type="fixed">
+  <parent link="camera_pole1"/>
+  <child link="camera_link1"/>
+  <origin xyz="0 0 1.04" rpy="0 0.785 3.925"/>
+</joint>
+<joint name="pole_to_camera2" type="fixed">
+  <parent link="camera_pole2"/>
+  <child link="camera_link2"/>
+  <origin xyz="0 0 1.04" rpy="0 0.785 0.785"/>
+</joint>
+<gazebo reference="camera_link1">
+  <sensor name="external_camera1" type="camera">
+    <topic>camera1/image_raw</topic> <camera>
       <horizontal_fov>1.089</horizontal_fov>
       <image>
         <width>1280</width>
         <height>720</height>
-        <format>R8G8B8</format>
       </image>
     </camera>
@@ -331,12 +340,18 @@
     <update_rate>30</update_rate>
     <visualize>true</visualize>
-    <plugin name="camera_controller" filename="libgazebo_ros_camera.so">
-      <alwaysOn>true</alwaysOn>
-      <updateRate>0.0</updateRate>
-      <cameraName>external_camera</cameraName>
-      <imageTopicName>image_raw</imageTopicName>
-      <cameraInfoTopicName>camera_info</cameraInfoTopicName>
-      <frameName>camera_link</frameName>
-    </plugin>
+  </sensor>
+</gazebo>
+<gazebo reference="camera_link2">
+  <sensor name="external_camera2" type="camera">
+    <topic>camera2/image_raw</topic> <camera>
+      <horizontal_fov>1.089</horizontal_fov>
+      <image>
+        <width>1280</width>
+        <height>720</height>
+      </image>
+    </camera>
+    <always_on>1</always_on>
+    <update_rate>30</update_rate>
+    <visualize>true</visualize>
   </sensor>
 </gazebo>
