Commit message: camera working

File: hcr5_ws/src/hcr5_description/urdf/hcr5.xacro (robot description, xacro)
@@ -244,4 +244,9 @@
   <plugin filename="gz_ros2_control-system" name="gz_ros2_control::GazeboSimROS2ControlPlugin">
     <parameters>$(find hcr5_description)/config/hcr5_controllers.yaml</parameters>
+  </plugin>
+  <plugin
+    filename="gz-sim-sensors-system"
+    name="gz::sim::systems::Sensors">
+    <render_engine>ogre2</render_engine>
   </plugin>
 </gazebo>
@@ -258,26 +263,20 @@
   <joint name="camera_joint" type="fixed">
     <parent link="link6_1"/> <child link="camera_link"/>
-    <origin xyz="-0.053 0.0 0.0" rpy="1.5708 1.5708 1.5708"/>
-  </joint>
-  <gazebo reference="camera_link">
-    <sensor name="robot_camera" type="camera">
-      <pose>0 0 0 0 0 0</pose>
-      <visualize>true</visualize>
-      <update_rate>30.0</update_rate>
-      <camera>
-        <horizontal_fov>1.089</horizontal_fov>
-        <image>
-          <width>640</width>
-          <height>480</height>
-          <format>R8G8B8</format>
-        </image>
-        <clip>
-          <near>0.05</near>
-          <far>8.0</far>
-        </clip>
-      </camera>
-      <topic>camera/image_raw</topic>
-      <gz_frame_id>camera_link</gz_frame_id>
-    </sensor>
-  </gazebo>
+    <origin xyz="-0.053 0.0 0.0" rpy="3.14159 3.14159 0.0"/>
+  </joint>
+<gazebo reference="camera_link">
+  <sensor name="robot_camera" type="camera">
+    <topic>camera/image_raw</topic>
+    <camera>
+      <horizontal_fov>1.089</horizontal_fov>
+      <image>
+        <width>640</width>
+        <height>480</height>
+      </image>
+    </camera>
+    <always_on>1</always_on>
+    <update_rate>30</update_rate>
+    <visualize>true</visualize>
+  </sensor>
+</gazebo>
 </robot>

Commit message: Enhance HCR5 functionality: add target cube link, update camera calibration, and implement motion controller and picker nodes

File: hcr5_ws/src/hcr5_description/urdf/hcr5.xacro (robot description, xacro)
@@ -31,4 +31,15 @@
   <child link="base_link"/>
   <origin xyz="0.195 -0.31 0.395" rpy="0 0 0.785"/>
+</joint>
+<link name="target_cube">
+  <visual>
+    <geometry><box size="0.04 0.04 0.04"/></geometry>
+    <material name="purple"><color rgba="0.5 0 0.5 1"/></material>
+  </visual>
+</link>
+<joint name="world_to_target" type="fixed">
+  <parent link="base_link"/>
+  <child link="target_cube"/>
+  <origin xyz="0.2 0.6 0.02" rpy="0 0 0"/>
 </joint>
 <link name="base_link">
@@ -305,5 +316,5 @@
     <camera>
       <horizontal_fov>1.089</horizontal_fov>
-      <image><width>1920</width><height>1080</height></image>
+      <image><width>1280</width><height>720</height></image>
     </camera>
     <always_on>1</always_on>

Commit message: Update HCR5 configuration and add unified picker functionality: modify environment variables, add motion script, and adjust target cube position

File: hcr5_ws/src/hcr5_description/urdf/hcr5.xacro (robot description, xacro)
@@ -41,5 +41,5 @@
   <parent link="base_link"/>
   <child link="target_cube"/>
-  <origin xyz="0.2 0.6 0.02" rpy="0 0 0"/>
+  <origin xyz="0.6 0.3 0.02" rpy="0 0 0"/>
 </joint>
 <link name="base_link">

Commit message: Refactor hcr5_moveit_config package structure and add gripper controller
- Removed old launch files and replaced them with symbolic links to the source files.
- Updated hcr5_controllers.yaml to include a new gripper controller with appropriate gains and constraints.
- Modified hcr5.xacro to include the gripper model and its joints.
- Updated hcr5.srdf to define a new gripper group and its states (open and close).
- Changed the link name in HCR5UnifiedPicker to use the new tcp_link for position and orientation constraints.
- Added hcr5_gripper.xacro to define the gripper's structure and control interfaces.

File: hcr5_ws/src/hcr5_description/urdf/hcr5.xacro (robot description, xacro)
@@ -3,4 +3,5 @@
 <xacro:include filename="$(find hcr5_description)/urdf/materials.xacro" />
 <xacro:include filename="$(find hcr5_description)/urdf/hcr5.gazebo" />
+<xacro:include filename="$(find hcr5_description)/urdf/hcr5_gripper.xacro" />
 <xacro:arg name="use_mock_hardware" default="true" />
 <link name="world"/>
@@ -37,4 +38,7 @@
     <material name="purple"><color rgba="0.5 0 0.5 1"/></material>
   </visual>
+  <collision>
+    <geometry><box size="0.04 0.04 0.04"/></geometry>
+  </collision>
 </link>
 <joint name="world_to_target" type="fixed">
@@ -197,4 +201,11 @@
   </collision>
 </link>
+<xacro:hcr5_gripper parent="link6_1" prefix="" />
+<link name="tcp_link"/>
+<joint name="gripper_to_tcp" type="fixed">
+  <parent link="gripper_base_link"/>
+  <child link="tcp_link"/>
+  <origin xyz="0 0 0.06" rpy="0 0 0"/>
+</joint>
 <joint name="joint_1" type="revolute">
   <origin xyz="0.0 0.0 0.03" rpy="0 0 0"/>
@@ -242,5 +253,5 @@
   <hardware>
     <xacro:if value="$(arg use_mock_hardware)">
-      <plugin>gz_ros2_control/GazeboSimSystem</plugin>
+      <plugin>ign_ros2_control/IgnitionSystem</plugin>
     </xacro:if>
     <xacro:unless value="$(arg use_mock_hardware)">
@@ -295,4 +306,7 @@
     <material name="gray"><color rgba="0.5 0.5 0.5 1.0"/></material>
   </visual>
+  <collision>
+    <geometry><cylinder radius="0.02" length="2.45"/></geometry>
+  </collision>
 </link>
 <joint name="base_to_pole1" type="fixed">
@@ -306,8 +320,12 @@
     <material name="blue"><color rgba="0 0 1 1"/></material>
   </visual>
+  <collision>
+    <geometry><box size="0.1 0.1 0.1"/></geometry>
+  </collision>
 </link>
 <joint name="pole_to_camera1" type="fixed">
   <parent link="camera_pole1"/>
-  <child link="camera_link1"/> <origin xyz="0.05 -0.05 1.2" rpy="0 1.222 5.495"/> <!--rpy="0 70 315" degree-->
+  <child link="camera_link1"/>
+  <origin xyz="0.05 -0.05 1.2" rpy="0 1.222 5.495"/>
 </joint>
 <gazebo reference="camera_link1">
